File: switch/power.kicad_sch (KiCad schematic)
At the start: 13 parts, among them U2 LP2985-5.0

Commit message: Add case
Parts:
- F1: footprint Capacitor_THT:C_Disc_D8.0mm_W5.0mm_P5.00mm -> Fuse:Fuse_Littelfuse_395Series; MPN2 (none) -> Littelfuse:395-0100-0000
- U2: MPN1 (none) -> Texas Instruments:LP2985-50DBVR
Other:
- title: (none) -> IR-based AC switch

Commit message: Fix issues
Parts:
- C1: MPN (none) -> MKX2AW32205B00KSSD
- C3: MPN (none) -> 50SVPF68M
- D1: MPN (none) -> ABS6
- D2: MPN (none) -> MM1Z4734A
- F1: MPN (none) -> 395-0100-0000; MPN2 Littelfuse:395-0100-0000 -> (none)
- R4: MPN (none) -> CRF253-45T330R
- U2: MPN (none) -> LP2985-50DBVR
Changed lines of the file:
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@@
 			)
 		)
-		(property "MPN2" "Littelfuse:395-0100-0000"
+		(property "MPN" "395-0100-0000"
 			(at 43.18 50.8 90)
 			(effects
@@
 			)
 		)
+		(property "MPN" "MM1Z4734A"
+			(at 102.87 57.15 90)
+			(effects
+				(font
+					(size 1.27 1.27)
+				)
+				(hide yes)
+			)
+		)
 		(pin "2"
 		)
@@
 		)
 		(property "MPN1" "Diotec:ABS6"
+			(at 90.17 58.42 90)
+			(effects
+				(font
+					(size 1.27 1.27)
+				)
+				(hide yes)
+			)
+		)
+		(property "MPN" "ABS6"
 			(at 90.17 58.42 90)
 			(effects
@@
 			)
 		)
+		(property "MPN" "50SVPF68M"
+			(at 120.65 58.42 0)
+			(effects
+				(font
+					(size 1.27 1.27)
+				)
+				(hide yes)
+			)
+		)
 		(pin "1"
 		)
@@
 			)
 		)
+		(property "MPN" "MKX2AW32205B00KSSD"
+			(at 59.69 50.8 90)
+			(effects
+				(font
+					(size 1.27 1.27)
+				)
+				(hide yes)
+			)
+		)
 		(pin "1"
 		)
@@
 			)
 		)
+		(property "MPN" "LP2985-50DBVR"
+			(at 147.32 53.34 0)
+			(effects
+				(font
+					(size 1.27 1.27)
+				)
+				(hide yes)
+			)
+		)
 		(pin "3"
 		)
@@
 			(at 77.47 58.42 90)
 			(effects
+				(font
+					(size 1.27 1.27)
+				)
+				(hide yes)
+			)
+		)
+		(property "MPN" "CRF253-45T330R"
+			(at 77.47 58.42 90)
+			(effects
