File: switch/sense.kicad_sch (KiCad schematic)
At the start: 3 parts, among them Q1 DMG2305UX

Commit message: Add case
Parts:
- A1: MPN1 (none) -> Vishay:TSSP4038
Other:
- title: (none) -> IR-based AC switch

Commit message: Fix issues
Parts:
- A1: MP TSSP4038 -> (none); MPN (none) -> TSSP4038
- Q1: MPN (none) -> DMG2305UX-13
Changed lines of the file:
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@@
 			)
 		)
-		(property "MP" "TSSP4038"
+		(property "MPN" "TSSP4038"
 			(at 80.01 55.88 0)
 			(effects
@@
 			(at 118.11 55.88 0)
 			(effects
+				(font
+					(size 1.27 1.27)
+				)
+				(hide yes)
+			)
+		)
+		(property "MPN" "DMG2305UX-13"
+			(at 118.11 55.88 0)
+			(effects
