File: switch/switch.kicad_pcb (KiCad board)
At the start: 2 copper layers, 35.3 x 35.3 mm, 28 parts, among them J1 1935174, J2 1935174, K1 ASO242, Q1 SFH309, Q2 BC847

Commit message: Updated rev
Parts:
- removed C2: 68u, Capacitor_SMD:CP_Elec_10x12.5
- removed D3: Z1SMA12, Diode_SMD:D_SMA
- removed D5, D6: 1N4148WS, Diode_SMD:D_SOD-323_HandSoldering
- removed Q2: BC847, Package_TO_SOT_SMD:SOT-23
- removed R6: 10k, Resistor_SMD:R_0805_2012Metric
- added A1: TSSP4038, switch:XDCR_TSSP4038, F.Cu at (91.9, 66.2)
- added H4: MountingHole, MountingHole:MountingHole_2.2mm_M2_DIN965, F.Cu at (87.6, 69.5)
- added U2: LP2985-5.0, Package_TO_SOT_SMD:SOT-23-5, F.Cu at (92.0, 60.7)
- C1: value 330n -> 220nF; footprint Capacitor_THT:C_Rect_L24.0mm_W7.0mm_P22.50mm_MKT -> Capacitor_THT:C_Rect_L18.0mm_W8.0mm_P15.00mm_FKS3_FKP3
- C3: value 22u -> 68u; footprint Capacitor_SMD:C_1210_3225Metric -> Capacitor_SMD:CP_Elec_10x12.5
- C4: value 0.1u -> 1u; moved to F.Cu
- C5: value 0.1u -> 10nF; footprint Capacitor_SMD:C_0603_1608Metric -> Capacitor_SMD:C_0805_2012Metric; moved to F.Cu
- C6: value 22u -> 2.2uF; footprint Capacitor_SMD:C_1210_3225Metric -> Capacitor_SMD:C_0805_2012Metric
- D1: value 1N4148WS -> ABS6; footprint Diode_SMD:D_SOD-323_HandSoldering -> Diode_SMD:Diode_Bridge_Diotec_ABS; moved to F.Cu
- D2: value 1N4148WS -> MM1Z4734A; footprint Diode_SMD:D_SOD-323_HandSoldering -> Diode_SMD:D_SOD-123F; moved to F.Cu
- Q1: value SFH309 -> DMG2305UX; footprint LED_THT:LED_D3.0mm_Clear -> Package_TO_SOT_SMD:SOT-23; moved to B.Cu
- R1: value 330 -> 470k; footprint Resistor_THT:R_Axial_DIN0516_L15.5mm_D5.0mm_P7.62mm_Vertical -> Resistor_SMD:R_0805_2012Metric_Pad1.20x1.40mm_HandSolder; moved to B.Cu
- R2, R3: value 100k -> 470k; footprint Resistor_SMD:R_0805_2012Metric -> Resistor_SMD:R_0805_2012Metric_Pad1.20x1.40mm_HandSolder
- R4: value 100k -> 330; footprint Resistor_SMD:R_0805_2012Metric -> Resistor_THT:R_Axial_DIN0516_L15.5mm_D5.0mm_P7.62mm_Vertical; moved to F.Cu
- R5: value 0 -> 100k; footprint Resistor_SMD:R_0603_1608Metric -> Resistor_SMD:R_0805_2012Metric; moved to B.Cu
- moved REF** 32.9 mm to (105.8, 68.0)
- moved D2 21.2 mm to (112.1, 68.5), turned to 0 degrees
- moved D1 15.7 mm to (112.0, 62.9)
- moved REF** 14.8 mm to (106.1, 61.5)
- moved C3 14.7 mm to (102.3, 65.1), turned to 180 degrees
- moved R1 12.5 mm to (107.4, 50.0), turned to 0 degrees
- moved R5 12.3 mm to (91.9, 68.5), turned to 180 degrees
- moved H3 12.1 mm to (118.3, 69.5)
- moved R4 7.73 mm to (117.6, 58.2), turned to -90 degrees
- moved C4 7.04 mm to (94.8, 59.9), turned to -90 degrees
- moved Q1 5.88 mm to (92.0, 62.6), turned to -90 degrees
- moved C5 4.80 mm to (89.8, 58.0), turned to 180 degrees
- moved R3 4.41 mm to (107.4, 53.0), turned to 0 degrees
- moved R2 4.01 mm to (107.4, 51.5), turned to 180 degrees
- moved C6 3.33 mm to (88.9, 60.8), turned to 90 degrees
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Connections:
- net Net-(D1-A) renamed GND
- C3 pad 1: Net-(Q3-E) -> +5VA
- C4 pad 1: Net-(Q3-E) -> +5VA
- C5 pad 1: Net-(Q3-E) -> Net-(U2-BP)
- C6 pad 1: Net-(Q3-E) -> +5V
- D1 pad 1: Net-(D1-K) -> +5VA
- D2 pad 1: /N -> +5VA
- K1 pad 3: Net-(K1-+) -> /IR receiver/SWITCH
- Q1 pad 1: Net-(D3-K) -> Net-(A1-OUT)
- Q1 pad 2: Net-(Q1-E) -> +5V
- R1 pad 1: Net-(C1-Pad2) -> Net-(C1-Pad1)
- R1 pad 2: Net-(D1-K) -> Net-(R1-Pad2)
- R2 pad 1: Net-(C1-Pad1) -> Net-(R1-Pad2)
- R3 pad 2: Net-(R3-Pad2) -> Net-(C1-Pad2)
- R4 pad 1: Net-(R3-Pad2) -> Net-(C1-Pad2)
- R4 pad 2: Net-(C1-Pad2) -> Net-(D1-Pad4)
- R5 pad 1: Net-(Q3-E) -> +5V
- R5 pad 2: Net-(K1-+) -> Net-(A1-OUT)
Routing:
- net GND: track 46.4 -> 0.05 mm, vias 2 -> 0
- net Net-(D3-K): track 31.6 -> 0.00 mm, vias 1 -> 0
- net +5VA: track 0.00 -> 26.5 mm
- net Net-(D1-K): track 19.9 -> 0.00 mm
- net +5V: track 0.00 -> 18.7 mm
- net Net-(Q3-E): track 17.8 -> 0.00 mm, vias 1 -> 0
- net /IR receiver/SWITCH: track 0.00 -> 14.6 mm
- net Net-(D1-Pad4): track 0.00 -> 11.3 mm
- net Net-(A1-OUT): track 0.00 -> 8.23 mm
- net Net-(K1-+): track 5.74 -> 0.00 mm
- net Net-(Q1-E): track 5.64 -> 0.00 mm
- net /L_LOAD: track 19.2 -> 24.4 mm
- net /N: track 40.8 -> 35.8 mm
- net Net-(C1-Pad1): track 18.4 -> 14.2 mm
- net Net-(R3-Pad2): track 2.00 -> 0.00 mm
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- added copper zone on B.Cu, net GND
- added copper zone on F.Cu, net GND
- removed copper zone on B.Cu, net (none)
- removed copper zone on F.Cu, net (none)
Other:
- board size 35.3 x 35.3 mm -> 35.3 x 36.9 mm

Commit message: Add case
Parts:
- removed REF**: KiCad-Logo2_5mm_SilkScreen, Symbol:KiCad-Logo2_5mm_SilkScreen
- removed REF**: OSHW-Logo2_7.3x6mm_SilkScreen, Symbol:OSHW-Logo2_7.3x6mm_SilkScreen
- F1: footprint Capacitor_THT:C_Disc_D8.0mm_W5.0mm_P5.00mm -> Fuse:Fuse_Littelfuse_395Series
- H1, H2, H3, H4: footprint MountingHole:MountingHole_2.2mm_M2_DIN965 -> MountingHole:MountingHole_2.2mm_M2_ISO14580
- Q1, R5: moved to F.Cu
- moved C6 6.02 mm to (93.8, 64.3), turned to 180 degrees
- moved R5 5.53 mm to (88.1, 64.6)
- moved C5 5.49 mm to (91.0, 63.4), turned to -90 degrees
- moved A1 4.27 mm to (93.3, 70.2)
- moved Q1 3.95 mm to (88.1, 61.7), turned to 90 degrees
- moved C4 2.48 mm to (92.9, 58.3), turned to 0 degrees
- moved U2 1.76 mm to (93.7, 61.2), turned to -90 degrees
Routing:
- net +5VA: track 26.5 -> 30.4 mm
- net Net-(A1-OUT): track 8.23 -> 9.11 mm
- net +5V: track 18.7 -> 18.0 mm
- net GND: vias 0 -> 26

Commit message: Fix issues
Changed lines of the file:
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@@
 			(at 0 -2.9 0)
 			(layer "F.SilkS")
+			(hide yes)
 			(effects
 				(font
@@
 			)
 		)
+		(property "MPN" "LP2985-50DBVR"
+			(at 0 0 -90)
+			(unlocked yes)
+			(layer "F.Fab")
+			(hide yes)
+			(effects
+				(font
+					(size 1 1)
+					(thickness 0.15)
+				)
+			)
+		)
 		(property ki_fp_filters "SOT?23*")
 		(sheetname "Power")
@@
 			)
 		)
+		(property "MPN" "DMG2305UX-13"
+			(at 0 0 90)
+			(unlocked yes)
+			(layer "F.Fab")
+			(hide yes)
+			(effects
+				(font
+					(size 1 1)
+					(thickness 0.15)
+				)
+			)
+		)
 		(property ki_fp_filters "SOT?23*")
 		(sheetname "IR receiver")
@@
 			)
 		)
+		(property "MPN" "1935174"
+			(at 0 0 90)
+			(unlocked yes)
+			(layer "F.Fab")
+			(hide yes)
+			(effects
+				(font
+					(size 1 1)
+					(thickness 0.15)
+				)
+			)
+		)
 		(property ki_fp_filters "Connector*:*_1x??_*")
 		(sheetname "Root")
@@
 			)
 		)
-		(property "MP" "TSSP4038"
+		(property "PARTREV" "2.3"
 			(at 0 0 0)
 			(layer "F.Fab")
@@
 			)
 		)
-		(property "PARTREV" "2.3"
+		(property "Package" "None"
 			(at 0 0 0)
 			(layer "F.Fab")
@@
 			)
 		)
-		(property "Package" "None"
+		(property "Price" "None"
 			(at 0 0 0)
 			(layer "F.Fab")
@@
 			)
 		)
-		(property "Price" "None"
+		(property "Purchase-URL" "https://www.snapeda.com/api/url_track_click_mouser/?unipart_id=408177&manufacturer=Vishay Semiconductor&part_name=TSSP4038&search_term=None"
 			(at 0 0 0)
 			(layer "F.Fab")
@@
 			)
 		)
-		(property "Purchase-URL" "https://www.snapeda.com/api/url_track_click_mouser/?unipart_id=408177&manufacturer=Vishay Semiconductor&part_name=TSSP4038&search_term=None"
+		(property "STANDARD" "IPC 7351B"
 			(at 0 0 0)
 			(layer "F.Fab")
@@
 			)
 		)
-		(property "STANDARD" "IPC 7351B"
+		(property "SnapEDA_Link" "https://www.snapeda.com/parts/TSSP4038/Vishay+Semiconductor+Opto+Division/view-part/?ref=snap"
 			(at 0 0 0)
 			(layer "F.Fab")
@@
 			)
 		)
-		(property "SnapEDA_Link" "https://www.snapeda.com/parts/TSSP4038/Vishay+Semiconductor+Opto+Division/view-part/?ref=snap"
+		(property "MPN1" "Vishay:TSSP4038"
 			(at 0 0 0)
+			(unlocked yes)
 			(layer "F.Fab")
 			(hide yes)
@@
 			)
 		)
-		(property "MPN1" "Vishay:TSSP4038"
+		(property "MPN" "TSSP4038"
 			(at 0 0 0)
 			(unlocked yes)
@@
 			(at 0 -2.9 0)
 			(layer "F.SilkS")
+			(hide yes)
 			(effects
 				(font
@@
 			)
 		)
+		(property "MPN" "50SVPF68M"
+			(at 0 0 180)
+			(unlocked yes)
+			(layer "F.Fab")
+			(hide yes)
+			(effects
+				(font
+					(size 1 1)
+					(thickness 0.15)
+				)
+			)
+		)
 		(property ki_fp_filters "CP_*")
 		(sheetname "Power")
@@
 			)
 		)
+		(property "MPN" "1935174"
+			(at 0 0 -90)
+			(unlocked yes)
+			(layer "F.Fab")
+			(hide yes)
+			(effects
+				(font
+					(size 1 1)
+					(thickness 0.15)
+				)
+			)
+		)
 		(property ki_fp_filters "Connector*:*_1x??_*")
 		(sheetname "Root")
@@
 			)
 		)
+		(property "MPN" "CRF253-45T330R"
+			(at 0 0 -90)
+			(unlocked yes)
+			(layer "F.Fab")
+			(hide yes)
+			(effects
+				(font
+					(size 1 1)
+					(thickness 0.15)
+				)
+			)
+		)
 		(property ki_fp_filters "R_*")
 		(sheetname "Power")
@@
 			(at 0 -2.9 0)
 			(layer "F.SilkS")
+			(hide yes)
 			(effects
 				(font
@@
 			(at 0 -2.9 0)
 			(layer "F.SilkS")
+			(hide yes)
 			(effects
 				(font
@@
 			)
 		)
+		(property "MPN" "MKX2AW32205B00KSSD"
+			(at 0 0 -90)
+			(unlocked yes)
+			(layer "F.Fab")
+			(hide yes)
+			(effects
+				(font
+					(size 1 1)
+					(thickness 0.15)
+				)
+			)
+		)
 		(property ki_fp_filters "C_*")
 		(sheetname "Power")
@@
 			)
 		)
+		(property "MPN" "ABS6"
+			(at 0 0 90)
+			(unlocked yes)
+			(layer "F.Fab")
+			(hide yes)
+			(effects
+				(font
+					(size 1 1)
+					(thickness 0.15)
+				)
+			)
+		)
 		(property ki_fp_filters "Diode*Bridge*Diotec*ABS*")
 		(sheetname "Power")
@@
 			)
 		)
-		(property "MPN2" "Littelfuse:395-0100-0000"
+		(property "MPN" "395-0100-0000"
 			(at 0 0 0)
 			(unlocked yes)
@@
 			)
 		)
-		(property "Description" "\nFeatures ?DC Control, AC Output ?Triac (AO) or SCR (ASO) Output ?UL, CSA Approved ?Dimensions (L\n"
+		(property "Description" "Features ?DC Control, AC Output ?Triac (AO) or SCR (ASO) Output ?UL, CSA Approved ?Dimensions (L"
 			(at 51.20145 145.40145 0)
 			(layer "F.Fab")
@@
 			)
 		)
-		(property "MP" "ASO242"
+		(property "MPN1" "Sensata:ASO242"
 			(at 51.20145 145.40145 0)
 			(layer "F.Fab")
@@
 			)
 		)
-		(property "MPN1" "Sensata:ASO242"
+		(property "Package" "None"
 			(at 51.20145 145.40145 0)
 			(layer "F.Fab")
@@
 			)
 		)
-		(property "Package" "None"
+		(property "SKU1" "Conrad:188012"
 			(at 51.20145 145.40145 0)
 			(layer "F.Fab")
@@
 			)
 		)
-		(property "SKU1" "Conrad:188012"
+		(property "SnapEDA_Link" "https://www.snapeda.com/parts/ASO242/Crydom/view-part/?ref=snap"
 			(at 51.20145 145.40145 0)
 			(layer "F.Fab")
@@
 			)
 		)
-		(property "SnapEDA_Link" "https://www.snapeda.com/parts/ASO242/Crydom/view-part/?ref=snap"
-			(at 51.20145 145.40145 0)
+		(property "MPN" "ASO242"
+			(at 0 0 -90)
+			(unlocked yes)
 			(layer "F.Fab")
 			(hide yes)
@@
 			(layer "F.Fab")
 			(hide yes)
+			(effects
+				(font
+					(size 1 1)
+					(thickness 0.15)
+				)
+			)
+		)
+		(property "MPN" "MM1Z4734A"
+			(at 0 0 0)
+			(unlocked yes)
+			(layer "F.Fab")
+			(hide yes)
